File: cpod/layout/cpod-MCP1700-AM2321.brd (EAGLE design)
At the start: 12 parts

Commit message: 可以说是比较完美的一个布局
Routing:
- net N$1: track 208.3 -> 0.00 mm
- net GND: track 0.00 -> 81.9 mm
- net VCC: track 0.00 -> 55.3 mm
- net CSN: track 0.00 -> 43.4 mm
- net MISO: track 0.00 -> 34.1 mm
- net CE: track 0.00 -> 33.8 mm
- net MOSI: track 0.00 -> 27.8 mm
- net SCK: track 0.00 -> 20.2 mm
- net SCL: track 0.00 -> 13.8 mm
- net SDA: track 0.00 -> 11.2 mm
- net RAW: track 0.00 -> 11.2 mm
Changed lines of the file:
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@@
 <plain>
 <rectangle x1="0" y1="-43.18" x2="27.94" y2="0" layer="41"/>
+<wire x1="0" y1="0" x2="60.96" y2="0" width="0.4064" layer="41"/>
+<wire x1="60.96" y1="0" x2="60.96" y2="-43.18" width="0.4064" layer="41"/>
+<wire x1="60.96" y1="-43.18" x2="0" y2="-43.18" width="0.4064" layer="41"/>
+<wire x1="0" y1="-43.18" x2="0" y2="0" width="0.4064" layer="41"/>
 </plain>
 <attributes>
@@
 <contactref element="I2C" pad="2"/>
 <contactref element="R4" pad="P$1"/>
-<wire x1="41.91" y1="-29.21" x2="41.91" y2="-26.67" width="0" layer="19" extent="1-1"/>
-<wire x1="31.75" y1="-31.75" x2="41.91" y2="-29.21" width="0" layer="19" extent="1-1"/>
+<wire x1="34.29" y1="-29.21" x2="31.75" y2="-31.75" width="0.254" layer="16"/>
+<wire x1="41.91" y1="-29.21" x2="34.29" y2="-29.21" width="0.254" layer="16"/>
+<wire x1="41.91" y1="-29.21" x2="41.91" y2="-26.67" width="0.254" layer="1"/>
 </signal>
 <signal name="GND">
@@
 <contactref element="SUPPLY" pad="6"/>
 <contactref element="NRF24L01+" pad="1"/>
-<wire x1="59.69" y1="-26.67" x2="52.07" y2="-1.27" width="0" layer="19" extent="1-1"/>
-<wire x1="44.45" y1="-41.91" x2="59.69" y2="-26.67" width="0" layer="19" extent="1-1"/>
-<wire x1="41.91" y1="-41.91" x2="44.45" y2="-41.91" width="0" layer="19" extent="1-1"/>
-<wire x1="39.37" y1="-41.91" x2="41.91" y2="-41.91" width="0" layer="19" extent="1-1"/>
-<wire x1="36.83" y1="-41.91" x2="39.37" y2="-41.91" width="0" layer="19" extent="1-1"/>
-<wire x1="34.29" y1="-41.91" x2="36.83" y2="-41.91" width="0" layer="19" extent="1-1"/>
-<wire x1="34.29" y1="-36.83" x2="34.29" y2="-41.91" width="0" layer="19" extent="1-1"/>
-<wire x1="34.29" y1="-34.29" x2="34.29" y2="-36.83" width="0" layer="19" extent="1-1"/>
-<wire x1="34.29" y1="-31.75" x2="34.29" y2="-34.29" width="0" layer="19" extent="1-1"/>
-<wire x1="36.83" y1="-36.83" x2="34.29" y2="-36.83" width="0" layer="19" extent="1-1"/>
+<wire x1="34.29" y1="-34.29" x2="34.29" y2="-36.83" width="0.254" layer="1"/>
+<wire x1="34.29" y1="-36.83" x2="36.83" y2="-36.83" width="0.254" layer="1"/>
+<wire x1="34.29" y1="-34.29" x2="34.29" y2="-31.75" width="0.254" layer="1"/>
+<wire x1="36.83" y1="-41.91" x2="34.29" y2="-41.91" width="0.254" layer="1"/>
+<wire x1="36.83" y1="-41.91" x2="39.37" y2="-41.91" width="0.254" layer="1"/>
+<wire x1="39.37" y1="-41.91" x2="41.91" y2="-41.91" width="0.254" layer="1"/>
+<wire x1="41.91" y1="-41.91" x2="44.45" y2="-41.91" width="0.254" layer="1"/>
+<wire x1="34.29" y1="-41.91" x2="34.29" y2="-36.83" width="0.254" layer="1"/>
+<wire x1="53.34" y1="-20.32" x2="58.42" y2="-25.4" width="0.254" layer="1"/>
+<wire x1="58.42" y1="-25.4" x2="59.69" y2="-26.67" width="0.254" layer="1"/>
+<wire x1="53.34" y1="-2.54" x2="53.34" y2="-20.32" width="0.254" layer="1"/>
+<wire x1="52.07" y1="-1.27" x2="53.34" y2="-2.54" width="0.254" layer="1"/>
+<wire x1="58.42" y1="-41.91" x2="44.45" y2="-41.91" width="0.254" layer="1"/>
+<wire x1="58.42" y1="-25.4" x2="58.42" y2="-41.91" width="0.254" layer="1"/>
 </signal>
 <signal name="SDA">
@@
 <contactref element="I2C" pad="1"/>
 <contactref element="R3" pad="P$1"/>
-<wire x1="44.45" y1="-29.21" x2="44.45" y2="-26.67" width="0" layer="19" extent="1-1"/>
-<wire x1="36.83" y1="-31.75" x2="44.45" y2="-29.21" width="0" layer="19" extent="1-1"/>
+<wire x1="38.1" y1="-30.48" x2="36.83" y2="-31.75" width="0.254" layer="16"/>
+<wire x1="43.18" y1="-30.48" x2="38.1" y2="-30.48" width="0.254" layer="16"/>
+<wire x1="44.45" y1="-29.21" x2="43.18" y2="-30.48" width="0.254" layer="16"/>
+<wire x1="44.45" y1="-29.21" x2="44.45" y2="-26.67" width="0.254" layer="1"/>
 </signal>
 <signal name="VCC">
@@
 <contactref element="NRF24L01+" pad="2"/>
 <contactref element="MCP1700T-3302-TO" pad="3"/>
-<wire x1="59.69" y1="-29.21" x2="52.07" y2="-16.51" width="0" layer="19" extent="1-1"/>
-<wire x1="44.45" y1="-36.83" x2="59.69" y2="-29.21" width="0" layer="19" extent="1-1"/>
-<wire x1="41.91" y1="-36.83" x2="44.45" y2="-36.83" width="0" layer="19" extent="1-1"/>
-<wire x1="44.45" y1="-39.37" x2="44.45" y2="-36.83" width="0" layer="19" extent="1-1"/>
-<wire x1="39.37" y1="-36.83" x2="41.91" y2="-36.83" width="0" layer="19" extent="1-1"/>
-<wire x1="39.37" y1="-34.29" x2="39.37" y2="-36.83" width="0" layer="19" extent="1-1"/>
-<wire x1="39.37" y1="-31.75" x2="39.37" y2="-34.29" width="0" layer="19" extent="1-1"/>
-<wire x1="41.91" y1="-39.37" x2="41.91" y2="-36.83" width="0" layer="19" extent="1-1"/>
-<wire x1="39.37" y1="-39.37" x2="39.37" y2="-36.83" width="0" layer="19" extent="1-1"/>
-<wire x1="36.83" y1="-39.37" x2="39.37" y2="-39.37" width="0" layer="19" extent="1-1"/>
+<wire x1="39.37" y1="-39.37" x2="36.83" y2="-39.37" width="0.254" layer="1"/>
+<wire x1="39.37" y1="-39.37" x2="41.91" y2="-39.37" width="0.254" layer="1"/>
+<wire x1="41.91" y1="-39.37" x2="44.45" y2="-39.37" width="0.254" layer="1"/>
+<wire x1="39.37" y1="-34.29" x2="39.37" y2="-36.83" width="0.254" layer="1"/>
+<wire x1="39.37" y1="-34.29" x2="39.37" y2="-31.75" width="0.254" layer="1"/>
+<wire x1="39.37" y1="-36.83" x2="41.91" y2="-36.83" width="0.254" layer="1"/>
+<wire x1="41.91" y1="-36.83" x2="44.45" y2="-36.83" width="0.254" layer="1"/>
+<wire x1="52.07" y1="-36.83" x2="59.69" y2="-29.21" width="0.254" layer="16"/>
+<wire x1="44.45" y1="-36.83" x2="52.07" y2="-36.83" width="0.254" layer="16"/>
+<wire x1="58.42" y1="-22.86" x2="52.07" y2="-16.51" width="0.254" layer="16"/>
+<wire x1="58.42" y1="-29.21" x2="58.42" y2="-22.86" width="0.254" layer="16"/>
+<wire x1="59.69" y1="-29.21" x2="58.42" y2="-29.21" width="0.254" layer="16"/>
+<wire x1="44.45" y1="-36.83" x2="44.45" y2="-39.37" width="0.254" layer="16"/>
 </signal>
 <signal name="RAW">
@@
 <contactref element="C1" pad="1"/>
 <contactref element="RAW" pad="1"/>
-<wire x1="31.75" y1="-36.83" x2="31.75" y2="-41.91" width="0" layer="19" extent="1-1"/>
-<wire x1="36.83" y1="-34.29" x2="31.75" y2="-36.83" width="0" layer="19" extent="1-1"/>
+<wire x1="31.75" y1="-41.91" x2="31.75" y2="-36.83" width="0.254" layer="1"/>
+<wire x1="35.56" y1="-35.56" x2="36.83" y2="-34.29" width="0.254" layer="16"/>
+<wire x1="33.02" y1="-35.56" x2="35.56" y2="-35.56" width="0.254" layer="16"/>
+<wire x1="31.75" y1="-36.83" x2="33.02" y2="-35.56" width="0.254" layer="16"/>
 </signal>
 <signal name="AD3">
@@
 <contactref element="ARDUINO1" pad="4"/>
 <contactref element="NRF24L01+" pad="5"/>
-<wire x1="39.37" y1="-16.51" x2="54.61" y2="-26.67" width="0" layer="19" extent="1-1"/>
+<wire x1="45.72" y1="-22.86" x2="39.37" y2="-16.51" width="0.254" layer="16"/>
+<wire x1="52.07" y1="-22.86" x2="45.72" y2="-22.86" width="0.254" layer="16"/>
+<wire x1="54.61" y1="-25.4" x2="52.07" y2="-22.86" width="0.254" layer="16"/>
+<wire x1="54.61" y1="-26.67" x2="54.61" y2="-25.4" width="0.254" layer="16"/>
 </signal>
 <signal name="MISO">
 <contactref element="ARDUINO1" pad="3"/>
 <contactref element="NRF24L01+" pad="7"/>
-<wire x1="36.83" y1="-16.51" x2="52.07" y2="-26.67" width="0" layer="19" extent="1-1"/>
+<wire x1="35.56" y1="-15.24" x2="36.83" y2="-16.51" width="0.254" layer="16"/>
+<wire x1="33.02" y1="-15.24" x2="35.56" y2="-15.24" width="0.254" layer="16"/>
+<wire x1="33.02" y1="-25.4" x2="33.02" y2="-15.24" width="0.254" layer="16"/>
+<wire x1="50.8" y1="-25.4" x2="33.02" y2="-25.4" width="0.254" layer="16"/>
+<wire x1="52.07" y1="-26.67" x2="50.8" y2="-25.4" width="0.254" layer="16"/>
 </signal>
 <signal name="MOSI">
 <contactref element="ARDUINO1" pad="2"/>
 <contactref element="NRF24L01+" pad="6"/>
-<wire x1="34.29" y1="-16.51" x2="54.61" y2="-29.21" width="0" layer="19" extent="1-1"/>
+<wire x1="41.91" y1="-24.13" x2="34.29" y2="-16.51" width="0.254" layer="16"/>
+<wire x1="52.07" y1="-24.13" x2="41.91" y2="-24.13" width="0.254" layer="16"/>
+<wire x1="53.34" y1="-25.4" x2="52.07" y2="-24.13" width="0.254" layer="16"/>
+<wire x1="53.34" y1="-29.21" x2="53.34" y2="-25.4" width="0.254" layer="16"/>
+<wire x1="54.61" y1="-29.21" x2="53.34" y2="-29.21" width="0.254" layer="16"/>
 </signal>
 <signal name="D10">
@@
 <contactref element="NRF24L01+" pad="4"/>
 <contactref element="ARDUINO2" pad="2"/>
-<wire x1="57.15" y1="-29.21" x2="34.29" y2="-1.27" width="0" layer="19" extent="1-1"/>
+<wire x1="55.88" y1="-27.94" x2="57.15" y2="-29.21" width="0.254" layer="1"/>
+<wire x1="45.72" y1="-27.94" x2="55.88" y2="-27.94" width="0.254" layer="1"/>
+<wire x1="45.72" y1="-12.7" x2="45.72" y2="-27.94" width="0.254" layer="1"/>
+<wire x1="34.29" y1="-1.27" x2="45.72" y2="-12.7" width="0.254" layer="1"/>
 </signal>
 <signal name="CE">
 <contactref element="NRF24L01+" pad="3"/>
 <contactref element="ARDUINO2" pad="3"/>
-<wire x1="57.15" y1="-26.67" x2="36.83" y2="-1.27" width="0" layer="19" extent="1-1"/>
+<wire x1="48.26" y1="-17.78" x2="57.15" y2="-26.67" width="0.254" layer="1"/>
+<wire x1="48.26" y1="-12.7" x2="48.26" y2="-17.78" width="0.254" layer="1"/>
+<wire x1="36.83" y1="-1.27" x2="48.26" y2="-12.7" width="0.254" layer="1"/>
 </signal>
 <signal name="D9">
@@
 <contactref element="NRF24L01+" pad="8"/>
 </signal>
-<signal name="N$1">
-<wire x1="0" y1="0" x2="60.96" y2="0" width="1.016" layer="16"/>
-<wire x1="60.96" y1="0" x2="60.96" y2="-43.18" width="1.016" layer="16"/>
-<wire x1="60.96" y1="-43.18" x2="0" y2="-43.18" width="1.016" layer="16"/>
-<wire x1="0" y1="-43.18" x2="0" y2="0" width="1.016" layer="16"/>
-</signal>
 </signals>

Commit message: 微调
Parts:
- added U$2: (no value), SparkFun-Aesthetics:OSHW-LOGO-L
Changed lines of the file:
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@@
 <element name="I2C" library="SparkFun-Connectors" package="1X02" value="" x="44.45" y="-26.67" rot="R180"/>
 <element name="SUPPLY" library="SparkFun-Connectors" package="2X4" value="M04X2" x="40.64" y="-40.64" rot="R180"/>
+<element name="U$2" library="SparkFun-Aesthetics" package="OSHW-LOGO-L" value="" x="5.08" y="-38.1"/>
 </elements>
 <signals>
